File: kicad_schematic_pcb/gps_gsm_prj.kicad_sch (KiCad schematic)
At the start: 16 parts, among them J1 USB_B, U1 LD1117S33TR_SOT223, U2 Pmod_GPS, U3 GSM_module

Commit message: documentation for project
Connections:
- net VU1_3V3: no longer A1.39 (VSYS), C5.1
- net Vin_5V: now also A1.39 (VSYS), C5.1
Changed lines of the file:
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@@
     (effects (font (size 1.27 1.27)) (justify left bottom))
   )
-  (label "VU1_3V3" (at 124.46 88.9 0)
+  (label "Vin_5V" (at 124.46 88.9 0)
     (effects (font (size 1.27 1.27)) (justify left bottom))
   )
@@
       (effects (font (size 1.27 1.27)) hide)
     )
+    (pin "2")
+    (pin "3")
+    (pin "5")
     (pin "6")
-    (pin "3")
-    (pin "2")
-    (pin "5")
   )
   (symbol (lib_id "power:GND1") (at 229.87 111.76 0) (unit 1)
@@
       (effects (font (size 1.27 1.27)) hide)
     )
-    (pin "8")
     (pin "12")
     (pin "13")
     (pin "14")
+    (pin "8")
   )
   (symbol (lib_id "T491A106K006AT:T491A106K006AT") (at 118.11 46.99 90) (unit 1)
